Commit message: Bee_mobile: Modified urdf to add real meshes, added missing links and joints, added a new node wheel_state_converter that converts wheel encoder angles that are of type Int64MultiArray to JointState, readable by RViz, configured the camera and the lidar in RViz, modified slam.launch.py to automatically configure and activate the slam_toolbox node with timers, started implementing odometry (does not currently work properly, WIP)

File: robot_ws/src/bee_mobile/urdf/robot.urdf.xacro (robot description, xacro)
@@ -1,60 +1,44 @@
 <?xml version="1.0"?>
 <robot name="four_wheel_robot" xmlns:xacro="http://www.ros.org/wiki/xacro">
+    <xacro:property name="pkg" value="package://bee_mobile/meshes" />
+    <!-- Position of the steering joint in the chassis frame of reference -->
+    <xacro:property name="front_x" value="0.5790" />
+    <xacro:property name="rear_x"  value="-0.5790" />
+    <xacro:property name="left_y"  value="-0.7661" />
+    <xacro:property name="right_y" value="0.1939" />
     <!-- Materials -->
-    <material name="blue">
-        <color rgba="0.0 0.5 0.8 1.0" />
+    <material name="black">
+        <color rgba="0.0 0.0 0.0 1.0" />
     </material>
-    <material name="dark_gray">
-        <color rgba="0.2 0.2 0.2 1.0" />
+    <material name="white">
+        <color rgba="1.0 1.0 1.0 1.0" />
     </material>
-    <material name="silver">
-        <color rgba="0.75 0.75 0.75 1.0" />
-    </material>
-    <material name="red">
-        <color rgba="0.8 0.1 0.1 1.0" />
-    </material>
-    <!-- Constants -->
-    <xacro:property name="M_PI" value="3.1415926535897931" />
-    <!-- Dimensions (meters) -->
-    <xacro:property name="chassis_length" value="1.4" />
-    <xacro:property name="chassis_width" value="1.0" />
-    <xacro:property name="chassis_depth" value="0.23" />
-    <xacro:property name="chassis_bottom_height" value="0.6" />
-    <xacro:property name="wheelbase" value="0.97" />
-    <xacro:property name="track_width" value="0.84" />
-    <xacro:property name="wheel_radius" value="0.215" />
-    <xacro:property name="wheel_thickness" value="0.2" />
-    <!-- Chassis centre (z = bottom + depth/2) -->
-    <xacro:property name="chassis_center_z" value="${chassis_bottom_height + chassis_depth/2}" />
-    <!-- Wheel positions -->
-    <xacro:property name="front_x" value="${wheelbase/2}" />
-    <xacro:property name="rear_x" value="${-wheelbase/2}" />
-    <xacro:property name="left_y" value="${-track_width/2}" />
-    <xacro:property name="right_y" value="${track_width/2}" />
-    <xacro:property name="wheel_z" value="${wheel_radius}" />
-    <!-- =========================== -->
-    <!-- Base Link (ground level)    -->
-    <!-- =========================== -->
+    <!-- Base Footprint - Virtual link representing the robot's 2D ground projection -->
+    <link name="base_footprint"/>
+    <joint name="base_footprint_joint" type="fixed">
+        <parent link="base_footprint"/>
+        <child link="base_link"/>
+        <origin xyz="0 0 0.8"/>
+    </joint>
     <link name="base_link" />
-    <!-- =========================== -->
-    <!-- Chassis                      -->
-    <!-- =========================== -->
+    <!-- Chassis -->
     <link name="chassis">
         <visual>
             <geometry>
-                <box size="${chassis_length} ${chassis_width} ${chassis_depth}" />
+                <mesh filename="${pkg}/chassis.STL" />
             </geometry>
-            <origin xyz="0 0 ${chassis_center_z}" rpy="0 0 0" />
-            <material name="blue" />
+            <origin xyz="0 0 0" rpy="0 0 0" />
+            <material name="white" />
         </visual>
         <collision>
             <geometry>
-                <box size="${chassis_length} ${chassis_width} ${chassis_depth}" />
+                <mesh filename="${pkg}/chassis.STL" />
             </geometry>
-            <origin xyz="0 0 ${chassis_center_z}" rpy="0 0 0" />
-        </collision>
-        <inertial>
-            <mass value="10.0" />
-            <inertia ixx="0.1" ixy="0.0" ixz="0.0" iyy="0.1" iyz="0.0" izz="0.1" />
+            <origin xyz="0 0 0" rpy="0 0 0" />
+        </collision>
+        <inertial>
+            <origin xyz="0.0079 -0.2513 -0.0925" rpy="0 0 0" />
+            <mass value="20.32" />
+            <inertia ixx="0.994429" ixy="0.000042" ixz="0.000001" iyy="0.520087" iyz="-0.001576" izz="1.481228" />
         </inertial>
     </link>
@@ -64,51 +48,268 @@
         <origin xyz="0 0 0" rpy="0 0 0" />
     </joint>
-    <!-- =========================== -->
-    <!-- Wheels (revolute joints)     -->
-    <!-- =========================== -->
-    <!-- Macro for a wheel -->
-    <xacro:macro name="wheel" params="name side x y">
+    <!-- ======= Wheel macro =======-->
+    <!-- name : front_left / front_right / rear_left / rear_right    -->
+    <!-- steering_joint_x/y : Position of the steering joint in the chassis frame of reference -->
+    <!-- steering_com_x/z : Center Of Mass position of the steering_link in its own frame of reference -->
+    <!-- wheel_joint_x : Position of the wheel_joint in the steering_link frame of reference -->
+    <!-- wheel_axis : Axis of the wheel_joint (-1 or 1) -->
+    <xacro:macro name="wheel" params="name steering_joint_x steering_joint_y steering_link_com_x steering_link_com_z wheel_joint_x wheel_axis">
+        <!-- Steering link -->
+        <link name="${name}_steering_link">
+            <visual>
+                <geometry>
+                    <mesh filename="${pkg}/${name}_steering_link.STL" />
+                </geometry>
+                <origin xyz="0 0 0" rpy="0 0 0" />
+                <material name="white" />
+            </visual>
+            <collision>
+                <geometry>
+                    <mesh filename="${pkg}/${name}_steering_link.STL" />
+                </geometry>
+                <origin xyz="0 0 0" rpy="0 0 0" />
+            </collision>
+            <inertial>
+                <origin xyz="${steering_link_com_x} 0 ${steering_link_com_z}" rpy="0 0 0" />
+                <mass value="0.88" />
+                <inertia ixx="0.002778" ixy="0.000001" ixz="0.000001" iyy="0.003568" iyz="0.000001" izz="0.001445" />
+            </inertial>
+        </link>
+        <!-- Steering joint -->
+        <joint name="${name}_steering_joint" type="revolute">
+            <parent link="chassis" />
+            <child link="${name}_steering_link" />
+            <origin xyz="${steering_joint_x} ${steering_joint_y} -0.2370" rpy="0 0 0" />
+            <axis xyz="0 0 1" />
+            <limit effort="100" velocity="5" lower="-1.5708" upper="1.5708" />
+            <dynamics damping="0.1" friction="0.1" />
+        </joint>
+        <!-- Wheel link -->
         <link name="${name}_link">
             <visual>
                 <geometry>
-                    <cylinder radius="${wheel_radius}" length="${wheel_thickness}" />
+                    <mesh filename="${pkg}/${name}_link.STL" />
                 </geometry>
-                <origin xyz="0 0 0" rpy="${M_PI/2} 0 0" /> <!-- rotate Z -> Y -->
-                <material name="dark_gray" />
+                <origin xyz="0 0 0" rpy="0 0 0" />
+                <material name="black" />
             </visual>
             <collision>
                 <geometry>
-                    <cylinder radius="${wheel_radius}" length="${wheel_thickness}" />
+                    <mesh filename="${pkg}/${name}_link.STL" />
                 </geometry>
-                <origin xyz="0 0 0" rpy="${M_PI/2} 0 0" />
+                <origin xyz="0 0 0" rpy="0 0 0" />
             </collision>
             <inertial>
-                <mass value="1.0" />
-                <inertia ixx="0.01" ixy="0" ixz="0" iyy="0.01" iyz="0" izz="0.01" />
+                <origin xyz="0 0 0" rpy="0 0 0" />
+                <mass value="12.84" />
+                <inertia ixx="0.280411" ixy="0.000001" ixz="0.000001" iyy="0.150110" iyz="0.000001" izz="0.150110" />
             </inertial>
         </link>
-        <joint name="${name}_joint" type="revolute">
-            <parent link="base_link" />
+        <!-- Wheel joint -->
+        <joint name="${name}_wheel_joint" type="continuous">
+            <parent link="${name}_steering_link" />
             <child link="${name}_link" />
-            <origin xyz="${x} ${y} ${wheel_z}" rpy="0 0 0" />
-            <axis xyz="0 1 0" /> <!-- rotation around Y -->
-            <limit effort="100" velocity="10" lower="-1e308" upper="1e308" />
+            <origin xyz="${wheel_joint_x} 0 -0.3505" rpy="0 0 0" />
+            <axis xyz="${wheel_axis} 0 0" />
             <dynamics damping="0.1" friction="0.1" />
         </joint>
     </xacro:macro>
-    <xacro:wheel name="front_left" side="left" x="${front_x}" y="${left_y}" />
-    <xacro:wheel name="front_right" side="right" x="${front_x}" y="${right_y}" />
-    <xacro:wheel name="rear_left" side="left" x="${rear_x}" y="${left_y}" />
-    <xacro:wheel name="rear_right" side="right" x="${rear_x}" y="${right_y}" />
-    <!-- =========================== -->
-    <!-- Camera & LiDAR (front centre, 0.83 m high) -->
-    <!-- =========================== -->
-    <link name="camera_link">
-        <visual>
-            <geometry>
-                <box size="0.1 0.1 0.07" />
-            </geometry>
+    <!-- Wheels -->
+    <xacro:wheel name="front_left" steering_joint_x="${front_x}" steering_joint_y="${left_y}" steering_link_com_x="0.0858"
+                 steering_link_com_z="-0.1461" wheel_joint_x="-0.0687" wheel_axis="-1" />
+    <xacro:wheel name="rear_left" steering_joint_x="${front_x}" steering_joint_y="${right_y}" steering_link_com_x="0.0858"
+                 steering_link_com_z="-0.1461" wheel_joint_x="-0.0687" wheel_axis="-1" />
+    <xacro:wheel name="front_right" steering_joint_x="${rear_x}" steering_joint_y="${left_y}" steering_link_com_x="-0.0858"
+                 steering_link_com_z="-0.1461" wheel_joint_x="0.0687" wheel_axis="1" />
+    <xacro:wheel name="rear_right" steering_joint_x="${rear_x}" steering_joint_y="${right_y}" steering_link_com_x="-0.0858"
+                 steering_link_com_z="-0.1461" wheel_joint_x="0.0687" wheel_axis="1" />
+    <!-- === Arm ===-->
+    <!-- Arm base slide (prismatic, X axis) -->
+    <link name="robot_arm_base_steering_link">
+        <visual>
+            <geometry><mesh filename="${pkg}/robot_arm_base_steering_link.STL" /></geometry>
+            <origin xyz="0 0 0" rpy="0 0 0" />
+            <material name="white" />
+        </visual>
+        <collision>
+            <geometry><mesh filename="${pkg}/robot_arm_base_steering_link.STL" /></geometry>
+        </collision>
+        <inertial>
+            <origin xyz="0 0.01577 0.0510" rpy="0 0 0" />
+            <mass value="1.539" />
+            <inertia ixx="0.00203" ixy="0.0" ixz="0.0" iyy="0.00238" iyz="0.0" izz="0.00328" />
+        </inertial>
+    </link>
+    <joint name="robot_arm_base_steering" type="prismatic">
+        <parent link="base_link" />
+        <child link="robot_arm_base_steering_link" />
+        <origin xyz="-0.186481 -0.233073 0.029" rpy="0 0 0" />
+        <axis xyz="1 0 0" />
+        <limit lower="-0.1" upper="0.38" effort="30" velocity="0.5" />
+    </joint>
+    <!-- Arm rotation (continuous, -Z axis) -->
+    <link name="robot_arm_steering_link">
+        <visual>
+            <geometry><mesh filename="${pkg}/robot_arm_steering_link.STL" /></geometry>
+            <origin xyz="0 0 0" rpy="0 0 0" />
+            <material name="white" />
+        </visual>
+        <collision>
+            <geometry><mesh filename="${pkg}/robot_arm_steering_link.STL" /></geometry>
+        </collision>
+        <inertial>
+            <origin xyz="-0.01159 0.02348 0.55969" rpy="0 0 0" />
+            <mass value="4.440" />
+            <inertia ixx="0.32071" ixy="0.0" ixz="0.0" iyy="0.32258" iyz="-0.00202" izz="0.00540" />
+        </inertial>
+    </link>
+    <joint name="robot_arm_steering_joint" type="continuous">
+        <parent link="robot_arm_base_steering_link" />
+        <child link="robot_arm_steering_link" />
+        <origin xyz="-0.026715 0.000282 0.072" rpy="0 0 0" />
+        <axis xyz="0 0 -1" />
+    </joint>
+    <!-- Vertical lift (prismatic, Z axis) -->
+    <link name="robot_arm_up_link">
+        <visual>
+            <geometry><mesh filename="${pkg}/robot_arm_up_link.STL" /></geometry>
+            <origin xyz="0 0 0" rpy="0 0 0" />
+            <material name="white" />
+        </visual>
+        <collision>
+            <geometry><mesh filename="${pkg}/robot_arm_up_link.STL" /></geometry>
+        </collision>
+        <inertial>
+            <origin xyz="-0.00475 -0.06999 -0.00710" rpy="0 0 0" />
+            <mass value="1.962" />
+            <inertia ixx="0.00593" ixy="0.0" ixz="0.0" iyy="0.00313" iyz="0.0" izz="0.00495" />
+        </inertial>
+    </link>
+    <joint name="robot_arm_up_joint" type="prismatic">
+        <parent link="robot_arm_steering_link" />
+        <child link="robot_arm_up_link" />
+        <origin xyz="-0.003162 -0.028282 0.172176" rpy="0 0 0" />
+        <axis xyz="0 0 1" />
+        <limit lower="-0.05" upper="1.0" effort="30" velocity="0.5" />
+    </joint>
+    <!-- Forward extension (prismatic, -Y axis) -->
+    <link name="robot_arm_front_link">
+        <visual>
+            <geometry><mesh filename="${pkg}/robot_arm_front_link.STL" /></geometry>
+            <origin xyz="0 0 0" rpy="0 0 0" />
+            <material name="white" />
+        </visual>
+        <collision>
+            <geometry><mesh filename="${pkg}/robot_arm_front_link.STL" /></geometry>
+        </collision>
+        <inertial>
+            <origin xyz="-0.02583 -0.03370 0.02627" rpy="0 0 0" />
+            <mass value="3.609" />
+            <inertia ixx="0.08333" ixy="0.0" ixz="0.0" iyy="0.04121" iyz="-0.00130" izz="0.04505" />
+        </inertial>
+    </link>
+    <joint name="robot_arm_front_joint" type="prismatic">
+        <parent link="robot_arm_up_link" />
+        <child link="robot_arm_front_link" />
+        <origin xyz="0.026377 -0.349803 -0.086735" rpy="0 0 0" />
+        <axis xyz="0 -1 0" />
+        <limit lower="0" upper="0.1" effort="30" velocity="0.5" />
+    </joint>
+    <!-- Vertical descent (prismatic, Z axis) -->
+    <link name="robot_arm_down_link">
+        <visual>
+            <geometry><mesh filename="${pkg}/robot_arm_down_link.STL" /></geometry>
+            <origin xyz="0 0 0" rpy="0 0 0" />
+            <material name="white" />
+        </visual>
+        <collision>
+            <geometry><mesh filename="${pkg}/robot_arm_down_link.STL" /></geometry>
+        </collision>
+        <inertial>
+            <origin xyz="0.00138 0.0 -0.00984" rpy="0 0 0" />
+            <mass value="0.924" />
+            <inertia ixx="0.00553" ixy="0.0" ixz="0.0" iyy="0.00446" iyz="0.0" izz="0.00137" />
+        </inertial>
+    </link>
+    <joint name="robot_arm_down_joint" type="prismatic">
+        <parent link="robot_arm_front_link" />
+        <child link="robot_arm_down_link" />
+        <origin xyz="-0.049 -0.029197 -0.027801" rpy="0 0 0" />
+        <axis xyz="0 0 1" />
+        <limit lower="-0.3" upper="0" effort="30" velocity="0.5" />
+    </joint>
+    <!-- Hand rotation (continuous, Z axis) -->
+    <link name="robot_hand_link">
+        <visual>
+            <geometry><mesh filename="${pkg}/robot_hand_link.STL" /></geometry>
+            <origin xyz="0 0 0" rpy="0 0 0" />
+            <material name="white" />
+        </visual>
+        <collision>
+            <geometry><mesh filename="${pkg}/robot_hand_link.STL" /></geometry>
+        </collision>
+        <inertial>
+            <origin xyz="-0.01395 -0.00114 0.01216" rpy="0 0 0" />
+            <mass value="0.245" />
+            <inertia ixx="0.00206" ixy="0.0" ixz="0.0" iyy="0.000230" iyz="0.0" izz="0.00227" />
+        </inertial>
+    </link>
+    <joint name="robot_hand_joint" type="continuous">
+        <parent link="robot_arm_down_link" />
+        <child link="robot_hand_link" />
+        <origin xyz="-0.010319 0 -0.244140" rpy="0 0 0" />
+        <axis xyz="0 0 1" />
+    </joint>
+    <!-- Finger 1 -->
+    <link name="finger_1_link">
+        <visual>
+            <geometry><mesh filename="${pkg}/finger_1_link.STL" /></geometry>
+            <origin xyz="0 0 0" rpy="0 0 0" />
+            <material name="white" />
+        </visual>
+        <collision>
+            <geometry><mesh filename="${pkg}/finger_1_link.STL" /></geometry>
+        </collision>
+        <inertial>
+            <origin xyz="0 0.0015 0" rpy="0 0 0" />
+            <mass value="0.00142" />
+            <inertia ixx="3.0e-7" ixy="0.0" ixz="0.0" iyy="3.5e-7" iyz="0.0" izz="4.8e-8" />
+        </inertial>
+    </link>
+    <joint name="finger_1_joint" type="continuous">
+        <parent link="robot_hand_link" />
+        <child link="finger_1_link" />
+        <origin xyz="-0.042813 -0.233796 0.014167" rpy="0 0 0" />
+        <axis xyz="0 -1 0" />
+    </joint>
+    <!-- Finger 2 -->
+    <link name="finger_2_link">
+        <visual>
+            <geometry><mesh filename="${pkg}/finger_2_link.STL" /></geometry>
+            <origin xyz="0 0 0" rpy="0 0 0" />
+            <material name="white" />
+        </visual>
+        <collision>
+            <geometry><mesh filename="${pkg}/finger_2_link.STL" /></geometry>
+        </collision>
+        <inertial>
+            <origin xyz="0.000723 -0.01025 -0.01093" rpy="0 0 0" />
+            <mass value="0.00145" />
+            <inertia ixx="3.0e-7" ixy="0.0" ixz="0.0" iyy="3.5e-7" iyz="0.0" izz="4.8e-8" />
+        </inertial>
+    </link>
+    <joint name="finger_2_joint" type="continuous">
+        <parent link="robot_hand_link" />
+        <child link="finger_2_link" />
+        <origin xyz="-0.016681 0.239546 0.025" rpy="0 0 0" />
+        <axis xyz="0 1 0" />
+    </joint>
+    <!-- === Sensors === -->
+    <!-- Camera -->
+    <link name="default_cam">
+        <visual>
+            <geometry><box size="0.1 0.1 0.07" /></geometry>
             <origin xyz="0 0 0" />
-            <material name="silver" />
+            <material name="white" />
         </visual>
         <inertial>
@@ -117,11 +318,15 @@
         </inertial>
     </link>
-    <link name="lidar_link">
-        <visual>
-            <geometry>
-                <cylinder radius="0.07" length="0.05" />
-            </geometry>
-            <origin xyz="0 0 0" rpy="0 0 0" />
-            <material name="silver" />
+    <joint name="camera_joint" type="fixed">
+        <parent link="base_link" />
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