Commit message: Bee_mobile : Fixed inertial (urdf) errors at display launch for the arm's fingers and changed orientations of the parts in the urdf file to have the positive x axis pointing in the forward direction (front of the robot), fixed topic naming error in the wheel_state_converter node and added a wheel position (integration of the speed) publisher, fixed an error linked to the timers of slam toolbox launch file causing it to crash, changed max_linear value in the joystick_node for testing, added small readme (build and launch), completely redesigned the odometry node, takes into acount the motor speed differences (front left slower) added a recalibration system (does not work properly, parameter fine tuning necessary)

File: robot_ws/src/bee_mobile/urdf/robot.urdf.xacro (robot description, xacro)
@@ -3,8 +3,8 @@
     <xacro:property name="pkg" value="package://bee_mobile/meshes" />
     <!-- Position of the steering joint in the chassis frame of reference -->
-    <xacro:property name="front_x" value="0.5790" />
-    <xacro:property name="rear_x"  value="-0.5790" />
-    <xacro:property name="left_y"  value="-0.7661" />
-    <xacro:property name="right_y" value="0.1939" />
+    <xacro:property name="left_y" value="0.5790" />
+    <xacro:property name="right_y"  value="-0.5790" />
+    <xacro:property name="front_x"  value="0.7661" />
+    <xacro:property name="rear_x" value="-0.1939" />
     <!-- Materials -->
     <material name="black">
@@ -16,10 +16,4 @@
     <!-- Base Footprint - Virtual link representing the robot's 2D ground projection -->
     <link name="base_footprint"/>
-    <joint name="base_footprint_joint" type="fixed">
-        <parent link="base_footprint"/>
-        <child link="base_link"/>
-        <origin xyz="0 0 0.8"/>
-    </joint>
-    <link name="base_link" />
     <!-- Chassis -->
     <link name="chassis">
@@ -28,5 +22,5 @@
                 <mesh filename="${pkg}/chassis.STL" />
             </geometry>
-            <origin xyz="0 0 0" rpy="0 0 0" />
+            <origin xyz="0 0 0" rpy="0 0 1.5708" />
             <material name="white" />
         </visual>
@@ -35,5 +29,5 @@
                 <mesh filename="${pkg}/chassis.STL" />
             </geometry>
-            <origin xyz="0 0 0" rpy="0 0 0" />
+            <origin xyz="0 0 0" rpy="0 0 1.5708" />
         </collision>
         <inertial>
@@ -43,8 +37,8 @@
         </inertial>
     </link>
-    <joint name="chassis_joint" type="fixed">
-        <parent link="base_link" />
-        <child link="chassis" />
-        <origin xyz="0 0 0" rpy="0 0 0" />
+    <joint name="base_footprint_joint" type="fixed">
+        <parent link="base_footprint"/>
+        <child link="chassis"/>
+        <origin xyz="0 0 0.8"/>
     </joint>
     <!-- ======= Wheel macro =======-->
@@ -54,5 +48,5 @@
     <!-- wheel_joint_x : Position of the wheel_joint in the steering_link frame of reference -->
     <!-- wheel_axis : Axis of the wheel_joint (-1 or 1) -->
-    <xacro:macro name="wheel" params="name steering_joint_x steering_joint_y steering_link_com_x steering_link_com_z wheel_joint_x wheel_axis">
+    <xacro:macro name="wheel" params="name steering_joint_x steering_joint_y steering_link_com_y steering_link_com_z wheel_joint_x wheel_axis">
         <!-- Steering link -->
         <link name="${name}_steering_link">
@@ -61,5 +55,5 @@
                     <mesh filename="${pkg}/${name}_steering_link.STL" />
                 </geometry>
-                <origin xyz="0 0 0" rpy="0 0 0" />
+                <origin xyz="0 0 0" rpy="0 0 1.5708" />
                 <material name="white" />
             </visual>
@@ -68,8 +62,8 @@
                     <mesh filename="${pkg}/${name}_steering_link.STL" />
                 </geometry>
-                <origin xyz="0 0 0" rpy="0 0 0" />
+                <origin xyz="0 0 0" rpy="0 0 1.5708" />
             </collision>
             <inertial>
-                <origin xyz="${steering_link_com_x} 0 ${steering_link_com_z}" rpy="0 0 0" />
+                <origin xyz="0 ${steering_link_com_y} ${steering_link_com_z}" rpy="0 0 0" />
                 <mass value="0.88" />
                 <inertia ixx="0.002778" ixy="0.000001" ixz="0.000001" iyy="0.003568" iyz="0.000001" izz="0.001445" />
@@ -91,6 +85,6 @@
                     <mesh filename="${pkg}/${name}_link.STL" />
                 </geometry>
-                <origin xyz="0 0 0" rpy="0 0 0" />
-                <material name="black" />
+                <origin xyz="0 0 0" rpy="0 0 1.5708" />
+                <material name="white" />
             </visual>
             <collision>
@@ -98,5 +92,5 @@
                     <mesh filename="${pkg}/${name}_link.STL" />
                 </geometry>
-                <origin xyz="0 0 0" rpy="0 0 0" />
+                <origin xyz="0 0 0" rpy="0 0 1.5708" />
             </collision>
             <inertial>
@@ -110,18 +104,18 @@
             <parent link="${name}_steering_link" />
             <child link="${name}_link" />
-            <origin xyz="${wheel_joint_x} 0 -0.3505" rpy="0 0 0" />
-            <axis xyz="${wheel_axis} 0 0" />
+            <origin xyz="0 ${wheel_joint_x} -0.3505" rpy="0 0 0" />
+            <axis xyz="0 ${wheel_axis} 0" />
             <dynamics damping="0.1" friction="0.1" />
         </joint>
     </xacro:macro>
     <!-- Wheels -->
-    <xacro:wheel name="front_left" steering_joint_x="${front_x}" steering_joint_y="${left_y}" steering_link_com_x="0.0858"
-                 steering_link_com_z="-0.1461" wheel_joint_x="-0.0687" wheel_axis="-1" />
-    <xacro:wheel name="rear_left" steering_joint_x="${front_x}" steering_joint_y="${right_y}" steering_link_com_x="0.0858"
-                 steering_link_com_z="-0.1461" wheel_joint_x="-0.0687" wheel_axis="-1" />
-    <xacro:wheel name="front_right" steering_joint_x="${rear_x}" steering_joint_y="${left_y}" steering_link_com_x="-0.0858"
-                 steering_link_com_z="-0.1461" wheel_joint_x="0.0687" wheel_axis="1" />
-    <xacro:wheel name="rear_right" steering_joint_x="${rear_x}" steering_joint_y="${right_y}" steering_link_com_x="-0.0858"
-                 steering_link_com_z="-0.1461" wheel_joint_x="0.0687" wheel_axis="1" />
+    <xacro:wheel name="front_left" steering_joint_x="${front_x}" steering_joint_y="${left_y}" steering_link_com_y="0.0858"
+                 steering_link_com_z="-0.1461" wheel_joint_x="-0.0687" wheel_axis="1" />
+    <xacro:wheel name="front_right" steering_joint_x="${front_x}" steering_joint_y="${right_y}" steering_link_com_y="0.0858"
+                 steering_link_com_z="-0.1461" wheel_joint_x="0.0687" wheel_axis="-1" />
+    <xacro:wheel name="rear_left" steering_joint_x="${rear_x}" steering_joint_y="${left_y}" steering_link_com_y="-0.0858"
+                 steering_link_com_z="-0.1461" wheel_joint_x="-0.0687" wheel_axis="1" />
+    <xacro:wheel name="rear_right" steering_joint_x="${rear_x}" steering_joint_y="${right_y}" steering_link_com_y="-0.0858"
+                 steering_link_com_z="-0.1461" wheel_joint_x="0.0687" wheel_axis="-1" />
     <!-- === Arm ===-->
     <!-- Arm base slide (prismatic, X axis) -->
@@ -129,5 +123,5 @@
         <visual>
             <geometry><mesh filename="${pkg}/robot_arm_base_steering_link.STL" /></geometry>
-            <origin xyz="0 0 0" rpy="0 0 0" />
+            <origin xyz="0 0 0" rpy="0 0 1.5708" />
             <material name="white" />
         </visual>
@@ -136,5 +130,5 @@
         </collision>
         <inertial>
-            <origin xyz="0 0.01577 0.0510" rpy="0 0 0" />
+            <origin xyz="0 0.01577 0.0510" rpy="0 0 1.5708" />
             <mass value="1.539" />
             <inertia ixx="0.00203" ixy="0.0" ixz="0.0" iyy="0.00238" iyz="0.0" izz="0.00328" />
@@ -142,8 +136,8 @@
     </link>
     <joint name="robot_arm_base_steering" type="prismatic">
-        <parent link="base_link" />
+        <parent link="chassis" />
         <child link="robot_arm_base_steering_link" />
-        <origin xyz="-0.186481 -0.233073 0.029" rpy="0 0 0" />
-        <axis xyz="1 0 0" />
+        <origin xyz="0.233073 -0.186481 0.029" rpy="0 0 0" />
+        <axis xyz="0 1 0" />
         <limit lower="-0.1" upper="0.38" effort="30" velocity="0.5" />
     </joint>
@@ -152,5 +146,5 @@
         <visual>
             <geometry><mesh filename="${pkg}/robot_arm_steering_link.STL" /></geometry>
-            <origin xyz="0 0 0" rpy="0 0 0" />
+            <origin xyz="0 0 0" rpy="0 0 1.5708" />
             <material name="white" />
         </visual>
@@ -159,5 +153,5 @@
         </collision>
         <inertial>
-            <origin xyz="-0.01159 0.02348 0.55969" rpy="0 0 0" />
+            <origin xyz="-0.01159 0.02348 0.55969" rpy="0 0 1.5708" />
             <mass value="4.440" />
             <inertia ixx="0.32071" ixy="0.0" ixz="0.0" iyy="0.32258" iyz="-0.00202" izz="0.00540" />
@@ -167,5 +161,5 @@
         <parent link="robot_arm_base_steering_link" />
         <child link="robot_arm_steering_link" />
-        <origin xyz="-0.026715 0.000282 0.072" rpy="0 0 0" />
+        <origin xyz="-0.000282 -0.026715 0.072" rpy="0 0 0" />
         <axis xyz="0 0 -1" />
     </joint>
@@ -174,5 +168,5 @@
         <visual>
             <geometry><mesh filename="${pkg}/robot_arm_up_link.STL" /></geometry>
-            <origin xyz="0 0 0" rpy="0 0 0" />
+            <origin xyz="0 0 0" rpy="0 0 1.5708" />
             <material name="white" />
         </visual>
@@ -181,5 +175,5 @@
         </collision>
         <inertial>
-            <origin xyz="-0.00475 -0.06999 -0.00710" rpy="0 0 0" />
+            <origin xyz="-0.00475 -0.06999 -0.00710" rpy="0 0 1.5708" />
             <mass value="1.962" />
             <inertia ixx="0.00593" ixy="0.0" ixz="0.0" iyy="0.00313" iyz="0.0" izz="0.00495" />
@@ -189,5 +183,5 @@
         <parent link="robot_arm_steering_link" />
         <child link="robot_arm_up_link" />
-        <origin xyz="-0.003162 -0.028282 0.172176" rpy="0 0 0" />
+        <origin xyz="0.028282 -0.003162 0.172176" rpy="0 0 0" />
         <axis xyz="0 0 1" />
         <limit lower="-0.05" upper="1.0" effort="30" velocity="0.5" />
@@ -197,5 +191,5 @@
         <visual>
             <geometry><mesh filename="${pkg}/robot_arm_front_link.STL" /></geometry>
-            <origin xyz="0 0 0" rpy="0 0 0" />
+            <origin xyz="0 0 0" rpy="0 0 1.5708" />
             <material name="white" />
         </visual>
@@ -204,5 +198,5 @@
         </collision>
         <inertial>
-            <origin xyz="-0.02583 -0.03370 0.02627" rpy="0 0 0" />
+            <origin xyz="-0.02583 -0.03370 0.02627" rpy="0 0 1.5708" />
             <mass value="3.609" />
             <inertia ixx="0.08333" ixy="0.0" ixz="0.0" iyy="0.04121" iyz="-0.00130" izz="0.04505" />
@@ -212,6 +206,6 @@
         <parent link="robot_arm_up_link" />
         <child link="robot_arm_front_link" />
-        <origin xyz="0.026377 -0.349803 -0.086735" rpy="0 0 0" />
-        <axis xyz="0 -1 0" />
+        <origin xyz="0.349803 0.026377 -0.086735" rpy="0 0 0" />
+        <axis xyz="1 0 0" />
         <limit lower="0" upper="0.1" effort="30" velocity="0.5" />
     </joint>
@@ -220,5 +214,5 @@
         <visual>
             <geometry><mesh filename="${pkg}/robot_arm_down_link.STL" /></geometry>
-            <origin xyz="0 0 0" rpy="0 0 0" />
+            <origin xyz="0 0 0" rpy="0 0 1.5708" />
             <material name="white" />
         </visual>
@@ -227,5 +221,5 @@
         </collision>
         <inertial>
-            <origin xyz="0.00138 0.0 -0.00984" rpy="0 0 0" />
+            <origin xyz="0.00138 0.0 -0.00984" rpy="0 0 1.5708" />
             <mass value="0.924" />
             <inertia ixx="0.00553" ixy="0.0" ixz="0.0" iyy="0.00446" iyz="0.0" izz="0.00137" />
@@ -235,5 +229,5 @@
         <parent link="robot_arm_front_link" />
         <child link="robot_arm_down_link" />
-        <origin xyz="-0.049 -0.029197 -0.027801" rpy="0 0 0" />
+        <origin xyz="0.029197 -0.049 -0.027801" rpy="0 0 0" />
         <axis xyz="0 0 1" />
         <limit lower="-0.3" upper="0" effort="30" velocity="0.5" />
@@ -243,5 +237,5 @@
         <visual>
             <geometry><mesh filename="${pkg}/robot_hand_link.STL" /></geometry>
-            <origin xyz="0 0 0" rpy="0 0 0" />
+            <origin xyz="0 0 0" rpy="0 0 1.5708" />
             <material name="white" />
         </visual>
@@ -250,5 +244,5 @@
         </collision>
         <inertial>
-            <origin xyz="-0.01395 -0.00114 0.01216" rpy="0 0 0" />
+            <origin xyz="-0.01395 -0.00114 0.01216" rpy="0 0 1.5708" />
             <mass value="0.245" />
             <inertia ixx="0.00206" ixy="0.0" ixz="0.0" iyy="0.000230" iyz="0.0" izz="0.00227" />
@@ -258,5 +252,5 @@
         <parent link="robot_arm_down_link" />
         <child link="robot_hand_link" />
-        <origin xyz="-0.010319 0 -0.244140" rpy="0 0 0" />
+        <origin xyz="0 -0.010319 -0.244140" rpy="0 0 0" />
         <axis xyz="0 0 1" />
     </joint>
@@ -265,5 +259,5 @@
         <visual>
             <geometry><mesh filename="${pkg}/finger_1_link.STL" /></geometry>
-            <origin xyz="0 0 0" rpy="0 0 0" />
+            <origin xyz="0 0 0" rpy="0 0 1.5708" />
             <material name="white" />
         </visual>
@@ -272,7 +266,6 @@
         </collision>
         <inertial>
-            <origin xyz="0 0.0015 0" rpy="0 0 0" />
-            <mass value="0.00142" />
-            <inertia ixx="3.0e-7" ixy="0.0" ixz="0.0" iyy="3.5e-7" iyz="0.0" izz="4.8e-8" />
+            <mass value="0.1"/>
+            <inertia ixx="0.001" ixy="0.0" ixz="0.0" iyy="0.001" iyz="0.0" izz="0.001"/>
         </inertial>
     </link>
@@ -280,6 +273,6 @@
         <parent link="robot_hand_link" />
         <child link="finger_1_link" />
-        <origin xyz="-0.042813 -0.233796 0.014167" rpy="0 0 0" />
-        <axis xyz="0 -1 0" />
+        <origin xyz="0.233796 -0.042813 0.014167" rpy="0 0 0" />
+        <axis xyz="1 0 0" />
     </joint>
     <!-- Finger 2 -->
@@ -287,5 +280,5 @@
         <visual>
             <geometry><mesh filename="${pkg}/finger_2_link.STL" /></geometry>
-            <origin xyz="0 0 0" rpy="0 0 0" />
+            <origin xyz="0 0 0" rpy="0 0 1.5708" />
             <material name="white" />
         </visual>
@@ -294,7 +287,6 @@
         </collision>
         <inertial>
-            <origin xyz="0.000723 -0.01025 -0.01093" rpy="0 0 0" />
-            <mass value="0.00145" />
-            <inertia ixx="3.0e-7" ixy="0.0" ixz="0.0" iyy="3.5e-7" iyz="0.0" izz="4.8e-8" />
+            <mass value="0.1"/>
+            <inertia ixx="0.001" ixy="0.0" ixz="0.0" iyy="0.001" iyz="0.0" izz="0.001"/>
         </inertial>
     </link>
@@ -302,6 +294,6 @@
         <parent link="robot_hand_link" />
         <child link="finger_2_link" />
-        <origin xyz="-0.016681 0.239546 0.025" rpy="0 0 0" />
-        <axis xyz="0 1 0" />
+        <origin xyz="-0.239546 -0.016681 0.025" rpy="0 0 0" />
+        <axis xyz="-1 0 0" />
     </joint>
     <!-- === Sensors === -->
@@ -319,7 +311,7 @@
     </link>
     <joint name="camera_joint" type="fixed">
-        <parent link="base_link" />
+        <parent link="chassis" />
         <child link="default_cam" />
-        <origin xyz="0 -0.975 0.03" rpy="0 0 0" />
+        <origin xyz="0.975 0 0.03" rpy="0 0 0" />
     </joint>
     <!-- Lidar -->
@@ -336,7 +328,7 @@
     </link>
     <joint name="lidar_joint" type="fixed">
-        <parent link="base_link" />
+        <parent link="chassis" />
         <child link="laser_frame" />
-        <origin xyz="0 -0.975 0.09" rpy="0 0 1.545" />
+        <origin xyz="0.975 0 0.09" rpy="0 0 3.06" />
     </joint>
 </robot>

Commit message: correction orientation lidar dans urdf

File: robot_ws/src/bee_mobile/urdf/robot.urdf.xacro (robot description, xacro)
@@ -330,5 +330,5 @@
         <parent link="chassis" />
         <child link="laser_frame" />
-        <origin xyz="0.975 0 0.09" rpy="0 0 3.06" />
+        <origin xyz="0.975 0 0.09" rpy="0 0 3.08" />
     </joint>
 </robot>

Commit message: sauvegarde code, etat actuel : nav2 marche pas totalement

File: robot_ws/src/bee_mobile/urdf/robot.urdf.xacro (robot description, xacro)
@@ -40,5 +40,5 @@
         <parent link="base_footprint"/>
         <child link="chassis"/>
-        <origin xyz="0 0 0.8"/>
+        <origin xyz="-0.2861 0 0.8"/>
     </joint>
     <!-- ======= Wheel macro =======-->
@@ -330,5 +330,5 @@
         <parent link="chassis" />
         <child link="laser_frame" />
-        <origin xyz="0.975 0 0.09" rpy="0 0 3.08" />
+        <origin xyz="0.975 0 0.09" rpy="0 0 3.0" />
     </joint>
 </robot>

Commit message: Feature: Séparation de l'odométrie du node de control car odométrie était calculée à partir des commandes et non des encodeurs, Implémentation de ros2_aruco, détection des tags aruco et publication de la TF dans un node qui s'abonne au topic aruco_markers, recalibration de la caméra assez précise (à quelques cm près)

File: robot_ws/src/bee_mobile/urdf/robot.urdf.xacro (robot description, xacro)
@@ -40,5 +40,5 @@
         <parent link="base_footprint"/>
         <child link="chassis"/>
-        <origin xyz="-0.2861 0 0.8"/>
+        <origin xyz="-0.2861 0 0.79"/>
     </joint>
     <!-- ======= Wheel macro =======-->
@@ -330,5 +330,5 @@
         <parent link="chassis" />
         <child link="laser_frame" />
-        <origin xyz="0.975 0 0.09" rpy="0 0 3.2" />
+        <origin xyz="0.975 0 0.09" rpy="0 0 3.08" />
     </joint>
 </robot>

Commit message: Feature: swerve_kinematics, réglage du problème de la vitesse minimale (robot galère à démarrer et ne s'arrête pas) :  suppression du mapping et des sauts de vitesse, remplacement par une courbe linéaire entre la vitesse calculée et la vitesse envoyée, et une portion concave sqrt entre 0.0 et la vitesse minimal 0.30m/s, modification des limites d'accélération dans nav2 params et swerve kinematics pour limiter les oscillations des commandes nav2 aux démarrage, modification du topic d'entrée nav2 du twist mux à /cmd_vel_nav car /cmd_vel_smoothed oscille beaucoup. résultats : le robot arrive bien à ses goals, démarre bien et s'arrête bien, mais deux problèmes encore : garde sa dernière vitesse après goal succeded donc on doit l'arrêter à la manette (R2) et dans les changements de direction, donne des vitesses aux roues alors qu'elles ne sont pas encore bien orientées => casse le robot

File: robot_ws/src/bee_mobile/urdf/robot.urdf.xacro (robot description, xacro)
@@ -330,5 +330,5 @@
         <parent link="chassis" />
         <child link="laser_frame" />
-        <origin xyz="0.975 0 0.09" rpy="0 0 3.08" />
+        <origin xyz="0.975 0 0.09" rpy="0 0 3.12" />
     </joint>
 </robot>

Commit message: Feature bee_mobile : modification de la courbe entre les vitesses calculées et les vitesses envoyées aux roues, montée en vitesse plus fluide, reste moins dans les basses vitesses qui génèrent des à-coups dans les roues, ajout d'une logique avant le slew rate et le mapping empéchant le robot d'avancer directement si les roues ne sont pas bien orientées (nécessaire car le mode omni de mppi considère que le robot peut tourner instantanément), plus les roues sont proches de leur angle cible, plus elle reçoivent de vitesse, facteur de vitesse appliqué à toutes les roues, calculé à partir de l'erreur la plus grande dans les 4 roues.

File: robot_ws/src/bee_mobile/urdf/robot.urdf.xacro (robot description, xacro)
@@ -330,5 +330,5 @@
         <parent link="chassis" />
         <child link="laser_frame" />
-        <origin xyz="0.975 0 0.09" rpy="0 0 3.12" />
+        <origin xyz="0.975 0 0.09" rpy="0 0 3.07" />
     </joint>
 </robot>

Commit message: correction bug caméra aruco, l'image compressed n'est pas bien détecté dans rviz et pas le node de détection de tag aruco, mais la fréquence est bonne sur pc portable et pc robot, avancement docking controller

File: robot_ws/src/bee_mobile/urdf/robot.urdf.xacro (robot description, xacro)
@@ -330,5 +330,5 @@
         <parent link="base_link" />
         <child link="laser_frame" />
-        <origin xyz="0.975 0 0.09" rpy="0 0 3.03" />
+        <origin xyz="0.975 0 0.09" rpy="0 0 3.06" />
     </joint>
 </robot>

Commit message: changements commit précédent

File: robot_ws/src/bee_mobile/urdf/robot.urdf.xacro (robot description, xacro)
@@ -332,3 +332,18 @@
         <origin xyz="0.975 0 0.09" rpy="0 0 3.06" />
     </joint>
+    <link name="gps_link">
+        <visual>
+        <geometry>
+            <cylinder radius="0.06" length="0.04"/>
+        </geometry>
+        <material name="black">
+            <color rgba="0.1 0.1 0.1 1.0"/>
+        </material>
+        </visual>
+    </link>
+    <joint name="gps_joint" type="fixed">
+        <parent link="base_link"/>
+        <child link="gps_link"/>
+        <origin xyz="0.2861 0.0 0.24" rpy="0.0 0.0 0.0"/>
+    </joint>
 </robot>
