Commit message: Bee_mobile : Simulation files, Waypoints commander to give the robot a series of 2d goal poses, twist_mux to merge (priority system) commands from nav2 and joystick which are then sent to the swerve controller, fixed an urdf model inconsistency (wheel separation = 0.96 in reality but in urdf = 1.158), reorganised the launch file and added a parameter for simulation (simulation:= True / False), tuned the pids and the nav2 params but they are still not perfect
Co-authored-by: Copilot <copilot@github.com>

File: robot_ws/src/bee_mobile/urdf/robot.urdf.xacro (robot description, xacro)
@@ -3,6 +3,6 @@
     <xacro:property name="pkg" value="package://bee_mobile/meshes" />
     <!-- Position of the steering joint in the chassis frame of reference -->
-    <xacro:property name="left_y" value="0.5790" />
-    <xacro:property name="right_y"  value="-0.5790" />
+    <xacro:property name="left_y" value="0.4150" /> <!-- 0.5790 -->
+    <xacro:property name="right_y"  value="-0.4150" /> <!-- -0.5790 -->
     <xacro:property name="front_x"  value="0.7661" />
     <xacro:property name="rear_x" value="-0.1939" />

Commit message: feature bee_mobile: ajustement de nombreux paramètres nav2 pour que le robot évite bien les obstacles, pour qu'il s'arrête correctement, et pour qu'il atteigne précisément ses objectifs, correction d'un bug d'odométrie dans le node swerve_kinematics_basic_test qui faisait tourner le robot légèrement à droite en avançant droit, et correction de la limite d'angle à 90 et -90 degrés, sécurité pour les à-coups pas encore ajoutée, modification de la carte pour tests pour simuler le passage étroit de 2m à la sortie de la zone de travail dans le labo
Co-authored-by: Copilot <copilot@github.com>

File: robot_ws/src/bee_mobile/urdf/robot.urdf.xacro (robot description, xacro)
@@ -32,5 +32,5 @@
         </collision>
         <inertial>
-            <origin xyz="0.0079 -0.2513 -0.0925" rpy="0 0 0" />
+            <origin xyz="0.2513 0.0 -0.0925" rpy="0 0 0" />
             <mass value="20.32" />
             <inertia ixx="0.994429" ixy="0.000042" ixz="0.000001" iyy="0.520087" iyz="-0.001576" izz="1.481228" />
@@ -130,5 +130,5 @@
         </collision>
         <inertial>
-            <origin xyz="0 0.01577 0.0510" rpy="0 0 1.5708" />
+            <origin xyz="-0.01577 0.0 0.0510" rpy="0 0 1.5708" />
             <mass value="1.539" />
             <inertia ixx="0.00203" ixy="0.0" ixz="0.0" iyy="0.00238" iyz="0.0" izz="0.00328" />
@@ -138,5 +138,5 @@
         <parent link="chassis" />
         <child link="robot_arm_base_steering_link" />
-        <origin xyz="0.233073 -0.186481 0.029" rpy="0 0 0" />
+        <origin xyz="0.233073 0.0 0.029" rpy="0 0 0" />
         <axis xyz="0 1 0" />
         <limit lower="-0.1" upper="0.38" effort="30" velocity="0.5" />
@@ -153,5 +153,5 @@
         </collision>
         <inertial>
-            <origin xyz="-0.01159 0.02348 0.55969" rpy="0 0 1.5708" />
+            <origin xyz="-0.02348 -0.01159 0.55969" rpy="0 0 1.5708" />
             <mass value="4.440" />
             <inertia ixx="0.32071" ixy="0.0" ixz="0.0" iyy="0.32258" iyz="-0.00202" izz="0.00540" />
@@ -175,5 +175,5 @@
         </collision>
         <inertial>
-            <origin xyz="-0.00475 -0.06999 -0.00710" rpy="0 0 1.5708" />
+            <origin xyz="0.06999 -0.00475 -0.00710" rpy="0 0 1.5708" />
             <mass value="1.962" />
             <inertia ixx="0.00593" ixy="0.0" ixz="0.0" iyy="0.00313" iyz="0.0" izz="0.00495" />
@@ -198,5 +198,5 @@
         </collision>
         <inertial>
-            <origin xyz="-0.02583 -0.03370 0.02627" rpy="0 0 1.5708" />
+            <origin xyz="0.03370 -0.02583 0.02627" rpy="0 0 1.5708" />
             <mass value="3.609" />
             <inertia ixx="0.08333" ixy="0.0" ixz="0.0" iyy="0.04121" iyz="-0.00130" izz="0.04505" />
@@ -221,5 +221,5 @@
         </collision>
         <inertial>
-            <origin xyz="0.00138 0.0 -0.00984" rpy="0 0 1.5708" />
+            <origin xyz="0.0 0.00138 -0.00984" rpy="0 0 1.5708" />
             <mass value="0.924" />
             <inertia ixx="0.00553" ixy="0.0" ixz="0.0" iyy="0.00446" iyz="0.0" izz="0.00137" />
@@ -244,5 +244,5 @@
         </collision>
         <inertial>
-            <origin xyz="-0.01395 -0.00114 0.01216" rpy="0 0 1.5708" />
+            <origin xyz="0.00114 -0.01395 0.01216" rpy="0 0 1.5708" />
             <mass value="0.245" />
             <inertia ixx="0.00206" ixy="0.0" ixz="0.0" iyy="0.000230" iyz="0.0" izz="0.00227" />

Commit message: Feature bee_mobile : Tests en réel avec nav2 et manette, problème de la vitesse min au démarage et à l'arrêt, ajustement de la vitesse min dans le node de control, ajustement pids, rajout de la préorientation des roues avec la manette en fonction du mode, ajustement params de vitesse dans nav2 params et aussi de précision du goal,
Co-authored-by: Copilot <copilot@github.com>

File: robot_ws/src/bee_mobile/urdf/robot.urdf.xacro (robot description, xacro)
@@ -330,5 +330,5 @@
         <parent link="chassis" />
         <child link="laser_frame" />
-        <origin xyz="0.975 0 0.09" rpy="0 0 3.0" />
+        <origin xyz="0.975 0 0.09" rpy="0 0 3.2" />
     </joint>
 </robot>

Commit message: Bee_mobile feature wip, ajout premiers fichiers pour gps et avancement sur la phase de docking
Co-authored-by: Copilot <copilot@github.com>

File: robot_ws/src/bee_mobile/urdf/robot.urdf.xacro (robot description, xacro)
@@ -330,5 +330,5 @@
         <parent link="chassis" />
         <child link="laser_frame" />
-        <origin xyz="0.975 0 0.09" rpy="0 0 3.07" />
+        <origin xyz="0.975 0 0.09" rpy="0 0 3.14" />
     </joint>
 </robot>

Commit message: Bee_mobile : avancement sur le docking, + mise en place du gps
Co-authored-by: Copilot <copilot@github.com>

File: robot_ws/src/bee_mobile/urdf/robot.urdf.xacro (robot description, xacro)
@@ -2,5 +2,5 @@
 <robot name="four_wheel_robot" xmlns:xacro="http://www.ros.org/wiki/xacro">
     <xacro:property name="pkg" value="package://bee_mobile/meshes" />
-    <!-- Position of the steering joint in the chassis frame of reference -->
+    <!-- Position of the steering joint in the base_link frame of reference -->
     <xacro:property name="left_y" value="0.4150" /> <!-- 0.5790 -->
     <xacro:property name="right_y"  value="-0.4150" /> <!-- -0.5790 -->
@@ -16,9 +16,9 @@
     <!-- Base Footprint - Virtual link representing the robot's 2D ground projection -->
     <link name="base_footprint"/>
-    <!-- Chassis -->
-    <link name="chassis">
+    <!-- Base_link (Chassis) -->
+    <link name="base_link">
         <visual>
             <geometry>
-                <mesh filename="${pkg}/chassis.STL" />
+                <mesh filename="${pkg}/base_link.STL" />
             </geometry>
             <origin xyz="0 0 0" rpy="0 0 1.5708" />
@@ -27,5 +27,5 @@
         <collision>
             <geometry>
-                <mesh filename="${pkg}/chassis.STL" />
+                <mesh filename="${pkg}/base_link.STL" />
             </geometry>
             <origin xyz="0 0 0" rpy="0 0 1.5708" />
@@ -39,10 +39,10 @@
     <joint name="base_footprint_joint" type="fixed">
         <parent link="base_footprint"/>
-        <child link="chassis"/>
+        <child link="base_link"/>
         <origin xyz="-0.2861 0 0.79"/>
     </joint>
     <!-- ======= Wheel macro =======-->
     <!-- name : front_left / front_right / rear_left / rear_right    -->
-    <!-- steering_joint_x/y : Position of the steering joint in the chassis frame of reference -->
+    <!-- steering_joint_x/y : Position of the steering joint in the base_link frame of reference -->
     <!-- steering_com_x/z : Center Of Mass position of the steering_link in its own frame of reference -->
     <!-- wheel_joint_x : Position of the wheel_joint in the steering_link frame of reference -->
@@ -72,5 +72,5 @@
         <!-- Steering joint -->
         <joint name="${name}_steering_joint" type="revolute">
-            <parent link="chassis" />
+            <parent link="base_link" />
             <child link="${name}_steering_link" />
             <origin xyz="${steering_joint_x} ${steering_joint_y} -0.2370" rpy="0 0 0" />
@@ -136,5 +136,5 @@
     </link>
     <joint name="robot_arm_base_steering" type="prismatic">
-        <parent link="chassis" />
+        <parent link="base_link" />
         <child link="robot_arm_base_steering_link" />
         <origin xyz="0.233073 0.0 0.029" rpy="0 0 0" />
@@ -311,5 +311,5 @@
     </link>
     <joint name="camera_joint" type="fixed">
-        <parent link="chassis" />
+        <parent link="base_link" />
         <child link="default_cam" />
         <origin xyz="0.975 0 0.03" rpy="0 0 0" />
@@ -328,7 +328,7 @@
     </link>
     <joint name="lidar_joint" type="fixed">
-        <parent link="chassis" />
+        <parent link="base_link" />
         <child link="laser_frame" />
-        <origin xyz="0.975 0 0.09" rpy="0 0 3.14" />
+        <origin xyz="0.975 0 0.09" rpy="0 0 3.03" />
     </joint>
 </robot>

Commit message: GPS : Simplification dans les TF caméra et base_link (plus d'offset par rapport au centre géométrique du robot), avancement sur la navigation gps, j'ai réussi à faire naviguer le robot mais pas précisemment car le signal sur gps est pas très qualitatif, à corriger
Co-authored-by: Copilot <copilot@github.com>

File: robot_ws/src/bee_mobile/urdf/robot.urdf.xacro (robot description, xacro)
@@ -5,6 +5,6 @@
     <xacro:property name="left_y" value="0.4150" /> <!-- 0.5790 -->
     <xacro:property name="right_y"  value="-0.4150" /> <!-- -0.5790 -->
-    <xacro:property name="front_x"  value="0.7661" />
-    <xacro:property name="rear_x" value="-0.1939" />
+    <xacro:property name="front_x"  value="0.48" /> <!-- 0.7661 -->
+    <xacro:property name="rear_x" value="-0.48" /> <!-- -0.1939 -->
     <!-- Materials -->
     <material name="black">
@@ -22,5 +22,5 @@
                 <mesh filename="${pkg}/base_link.STL" />
             </geometry>
-            <origin xyz="0 0 0" rpy="0 0 1.5708" />
+            <origin xyz="-0.2861 0 0" rpy="0 0 1.5708" />
             <material name="white" />
         </visual>
@@ -29,5 +29,5 @@
                 <mesh filename="${pkg}/base_link.STL" />
             </geometry>
-            <origin xyz="0 0 0" rpy="0 0 1.5708" />
+            <origin xyz="-0.2861 0 0" rpy="0 0 1.5708" />
         </collision>
         <inertial>
@@ -40,5 +40,5 @@
         <parent link="base_footprint"/>
         <child link="base_link"/>
-        <origin xyz="-0.2861 0 0.79"/>
+        <origin xyz="0 0 0.79"/>
     </joint>
     <!-- ======= Wheel macro =======-->
@@ -138,5 +138,5 @@
         <parent link="base_link" />
         <child link="robot_arm_base_steering_link" />
-        <origin xyz="0.233073 0.0 0.029" rpy="0 0 0" />
+        <origin xyz="-0.053027 0.0 0.029" rpy="0 0 0" />
         <axis xyz="0 1 0" />
         <limit lower="-0.1" upper="0.38" effort="30" velocity="0.5" />
@@ -299,8 +299,9 @@
     <!-- === Sensors === -->
     <!-- Camera -->
-    <link name="default_cam">
-        <visual>
-            <geometry><box size="0.1 0.1 0.07" /></geometry>
-            <origin xyz="0 0 0" />
+    <link name="camera_link">
+        <visual>
+            <geometry><box size="0.05 0.05 0.02" /></geometry>
+            <!-- <origin xyz="-0.081 0 0" rpy="1.5708 0.0 2.944"/> -->
+            <origin xyz="0 0 0" rpy="0 0 -0.05"/>
             <material name="white" />
         </visual>
@@ -311,7 +312,7 @@
     </link>
     <joint name="camera_joint" type="fixed">
-        <parent link="base_link" />
-        <child link="default_cam" />
-        <origin xyz="0.975 0 0.03" rpy="0 0 0" />
+        <parent link="base_link"/>
+        <child link="camera_link"/>
+        <origin xyz="0.7699 0.0 0.03" rpy="-2.0944 0.0 -1.5708"/> <!-- Rotation Roll (default : -pi/2 = -1.5708), Pitch, Yaw (caméra à -30 deg vers le bas -pi/2) en radians (REP-103) -->
     </joint>
     <!-- Lidar -->
@@ -330,5 +331,5 @@
         <parent link="base_link" />
         <child link="laser_frame" />
-        <origin xyz="0.975 0 0.09" rpy="0 0 3.06" />
+        <origin xyz="0.6889 0 0.09" rpy="0 0 3.06" />
     </joint>
     <link name="gps_link">
@@ -345,5 +346,5 @@
         <parent link="base_link"/>
         <child link="gps_link"/>
-        <origin xyz="0.2861 0.0 0.24" rpy="0.0 0.0 0.0"/>
+        <origin xyz="0 0.0 0.24" rpy="0.0 0.0 0.0"/>
     </joint>
 </robot>

Commit message: avancement gps nav, setup lidar
Co-authored-by: Copilot <copilot@github.com>

File: robot_ws/src/bee_mobile/urdf/robot.urdf.xacro (robot description, xacro)
@@ -317,5 +317,6 @@
     </joint>
     <!-- Lidar -->
-    <link name="laser_frame">
+    <!-- 1. Le capteur physique (Origine du nuage de points) -->
+    <link name="unilidar_lidar">
         <visual>
             <geometry><cylinder radius="0.07" length="0.05" /></geometry>
@@ -328,8 +329,19 @@
         </inertial>
     </link>
+    <!-- 2. Ancrage rigide du centre du Lidar sur le châssis -->
     <joint name="lidar_joint" type="fixed">
         <parent link="base_link" />
-        <child link="laser_frame" />
-        <origin xyz="0.6889 0 0.09" rpy="0 0 3.06" />
+        <child link="unilidar_lidar" />
+        <!-- Tes coordonnées de montage physique -->
+        <origin xyz="0.6889 0 0.09" rpy="0 0 0.45" />
+    </joint>
+    <!-- 3. Déclaration du repère de l'IMU interne -->
+    <link name="unilidar_imu" />
+    <!-- 4. Application stricte de la matrice de transformation Unitree -->
+    <!-- T_LI offset en mètres : X: -0.007698, Y: -0.014655, Z: 0.00667 -->
+    <joint name="lidar_to_imu_joint" type="fixed">
+        <parent link="unilidar_lidar" />
+        <child link="unilidar_imu" />
+        <origin xyz="-0.007698 -0.014655 0.00667" rpy="0 0 0" />
     </joint>
     <link name="gps_link">
@@ -346,5 +358,5 @@
         <parent link="base_link"/>
         <child link="gps_link"/>
-        <origin xyz="0.72 0.0 0.24" rpy="0.0 0.0 0.0"/>
+        <origin xyz="-0.72 0.0 0.24" rpy="0.0 0.0 0.0"/>
     </joint>
 </robot>

Commit message: Avancement sur algorithme swerve kinematics de control des moteurs,  indoor and outdoor configurations
Co-authored-by: Copilot <copilot@github.com>

File: robot_ws/src/bee_mobile/urdf/robot.urdf.xacro (robot description, xacro)
@@ -334,5 +334,5 @@
         <child link="unilidar_lidar" />
         <!-- Tes coordonnées de montage physique -->
-        <origin xyz="0.6889 0 0.09" rpy="0 0 0.45" />
+        <origin xyz="0.6889 0 0.09" rpy="1.5708 1.1208 1.5708" />
     </joint>
     <!-- 3. Déclaration du repère de l'IMU interne -->
@@ -343,5 +343,5 @@
         <parent link="unilidar_lidar" />
         <child link="unilidar_imu" />
-        <origin xyz="-0.007698 -0.014655 0.00667" rpy="0 0 0" />
+        <origin xyz="-0.007698 -0.014655 0.00667" rpy="0.0 0.0 0.0" />
     </joint>
     <link name="gps_link">
