Commit message: avancement gps nav, trajectoires ok, mais il faut toujours l'assister un peu pour ne pas qu'il rentre dans des murs, aussi souvent il y a une latence aux transitions des goals de la trajectoire, voir aussi pour le logiciel qgis

File: robot_ws/src/bee_mobile/urdf/robot.urdf.xacro (robot description, xacro)
@@ -346,5 +346,5 @@
         <parent link="base_link"/>
         <child link="gps_link"/>
-        <origin xyz="0 0.0 0.24" rpy="0.0 0.0 0.0"/>
+        <origin xyz="0.72 0.0 0.24" rpy="0.0 0.0 0.0"/>
     </joint>
 </robot>

Commit message: Tests en extérieurs, pas concluant car bug roue et pas assez de puissance que avec 2 roues et trucs encore à améliorer dans ackerman mode pour que ça marche, nécéssite plus de développement et de tests.

File: robot_ws/src/bee_mobile/urdf/robot.urdf.xacro (robot description, xacro)
@@ -120,5 +120,5 @@
     <!-- === Arm ===-->
     <!-- Arm base slide (prismatic, X axis) -->
-    <link name="robot_arm_base_steering_link">
+    <!-- <link name="robot_arm_base_steering_link">
         <visual>
             <geometry><mesh filename="${pkg}/robot_arm_base_steering_link.STL" /></geometry>
@@ -141,7 +141,7 @@
         <axis xyz="0 1 0" />
         <limit lower="-0.1" upper="0.38" effort="30" velocity="0.5" />
-    </joint>
+    </joint> -->
     <!-- Arm rotation (continuous, -Z axis) -->
-    <link name="robot_arm_steering_link">
+    <!-- <link name="robot_arm_steering_link">
         <visual>
             <geometry><mesh filename="${pkg}/robot_arm_steering_link.STL" /></geometry>
@@ -157,13 +157,13 @@
             <inertia ixx="0.32071" ixy="0.0" ixz="0.0" iyy="0.32258" iyz="-0.00202" izz="0.00540" />
         </inertial>
-    </link>
-    <joint name="robot_arm_steering_joint" type="continuous">
+    </link> -->
+    <!-- <joint name="robot_arm_steering_joint" type="continuous">
         <parent link="robot_arm_base_steering_link" />
         <child link="robot_arm_steering_link" />
         <origin xyz="-0.000282 -0.026715 0.072" rpy="0 0 0" />
         <axis xyz="0 0 -1" />
-    </joint>
+    </joint> -->
     <!-- Vertical lift (prismatic, Z axis) -->
-    <link name="robot_arm_up_link">
+    <!-- <link name="robot_arm_up_link">
         <visual>
             <geometry><mesh filename="${pkg}/robot_arm_up_link.STL" /></geometry>
@@ -186,7 +186,7 @@
         <axis xyz="0 0 1" />
         <limit lower="-0.05" upper="1.0" effort="30" velocity="0.5" />
-    </joint>
+    </joint> -->
     <!-- Forward extension (prismatic, -Y axis) -->
-    <link name="robot_arm_front_link">
+    <!-- <link name="robot_arm_front_link">
         <visual>
             <geometry><mesh filename="${pkg}/robot_arm_front_link.STL" /></geometry>
@@ -209,7 +209,7 @@
         <axis xyz="1 0 0" />
         <limit lower="0" upper="0.1" effort="30" velocity="0.5" />
-    </joint>
+    </joint> -->
     <!-- Vertical descent (prismatic, Z axis) -->
-    <link name="robot_arm_down_link">
+    <!-- <link name="robot_arm_down_link">
         <visual>
             <geometry><mesh filename="${pkg}/robot_arm_down_link.STL" /></geometry>
@@ -232,7 +232,7 @@
         <axis xyz="0 0 1" />
         <limit lower="-0.3" upper="0" effort="30" velocity="0.5" />
-    </joint>
+    </joint> -->
     <!-- Hand rotation (continuous, Z axis) -->
-    <link name="robot_hand_link">
+    <!-- <link name="robot_hand_link">
         <visual>
             <geometry><mesh filename="${pkg}/robot_hand_link.STL" /></geometry>
@@ -254,7 +254,7 @@
         <origin xyz="0 -0.010319 -0.244140" rpy="0 0 0" />
         <axis xyz="0 0 1" />
-    </joint>
+    </joint> -->
     <!-- Finger 1 -->
-    <link name="finger_1_link">
+    <!-- <link name="finger_1_link">
         <visual>
             <geometry><mesh filename="${pkg}/finger_1_link.STL" /></geometry>
@@ -275,7 +275,7 @@
         <origin xyz="0.233796 -0.042813 0.014167" rpy="0 0 0" />
         <axis xyz="1 0 0" />
-    </joint>
+    </joint> -->
     <!-- Finger 2 -->
-    <link name="finger_2_link">
+    <!-- <link name="finger_2_link">
         <visual>
             <geometry><mesh filename="${pkg}/finger_2_link.STL" /></geometry>
@@ -296,5 +296,5 @@
         <origin xyz="-0.239546 -0.016681 0.025" rpy="0 0 0" />
         <axis xyz="-1 0 0" />
-    </joint>
+    </joint> -->
     <!-- === Sensors === -->
     <!-- Camera -->

Commit message: docs: translate comments to english, add maintenance doc and finalize README - Translated code comments from French to English for better accessibility. - Added a maintenance documentation for future reference. - Completely rewritten and finalized the README.md with clear instructions and structure.

File: robot_ws/src/bee_mobile/urdf/robot.urdf.xacro (robot description, xacro)
@@ -314,8 +314,8 @@
         <parent link="base_link"/>
         <child link="camera_link"/>
-        <origin xyz="0.7699 0.0 0.03" rpy="-2.0944 0.0 -1.5708"/> <!-- Rotation Roll (default : -pi/2 = -1.5708), Pitch, Yaw (caméra à -30 deg vers le bas -pi/2) en radians (REP-103) -->
+        <origin xyz="0.7699 0.0 0.03" rpy="-2.0944 0.0 -1.5708"/> <!-- Roll, pitch, yaw rotation (camera tilted down by 30 degrees, -pi/2) in radians (REP-103). -->
     </joint>
     <!-- Lidar -->
-    <!-- 1. Le capteur physique (Origine du nuage de points) -->
+    <!-- 1. Physical sensor (point-cloud origin). -->
     <link name="unilidar_lidar">
         <visual>
@@ -329,15 +329,15 @@
         </inertial>
     </link>
-    <!-- 2. Ancrage rigide du centre du Lidar sur le châssis -->
+    <!-- 2. Rigid mounting of the LiDAR center on the chassis. -->
     <joint name="lidar_joint" type="fixed">
         <parent link="base_link" />
         <child link="unilidar_lidar" />
-        <!-- Tes coordonnées de montage physique -->
+        <!-- Physical mounting coordinates. -->
         <origin xyz="0.6889 0 0.09" rpy="1.5708 1.1208 1.5708" />
     </joint>
-    <!-- 3. Déclaration du repère de l'IMU interne -->
+    <!-- 3. Internal IMU frame declaration. -->
     <link name="unilidar_imu" />
-    <!-- 4. Application stricte de la matrice de transformation Unitree -->
-    <!-- T_LI offset en mètres : X: -0.007698, Y: -0.014655, Z: 0.00667 -->
+    <!-- 4. Strict application of the Unitree transformation matrix. -->
+    <!-- T_LI offset in meters: X: -0.007698, Y: -0.014655, Z: 0.00667 -->
     <joint name="lidar_to_imu_joint" type="fixed">
         <parent link="unilidar_lidar" />
